Commit message: Added joint spline action

File: iiwa_description/urdf/iiwa7.xacro (robot description, xacro)
@@ -189,5 +189,5 @@
       <origin xyz="0 0.21 0" rpy="${-PI / 2} ${PI} 0"/>
       <axis xyz="0 0 1"/>
-      <limit lower="${-170 * PI / 180}" upper="${170 * PI / 180}"
+      <limit lower="${-169 * PI / 180}" upper="${169 * PI / 180}"
              effort="${max_effort}" velocity="${max_velocity}" />
       <safety_controller soft_lower_limit="${-168 * PI / 180}"
